File: programming adapter/ATtiny 85 programming adapter/ATtiny 85 programming adapter.kicad_pcb (KiCad board)
At the start: 2 copper layers, 10 parts, among them J1 Conn_01x04_Male, J2 Conn_01x04_Male, J3 Conn_02x03_Odd_Even, J4 USB_B_Micro, SW1-Reset1 SW_Push, SW2-Power1 SW_SPST, U1 ATtiny85-20PU

Commit message: copyright note included, production data exported
Other:
- net class Default removed
