File: debugging boards/ATtiny85_default_debugging_board/ATtiny85_default_debugging_board.kicad_pcb (KiCad board)
At the start: 2 copper layers, 50.8 x 66 mm, 15 parts, among them J1 USB_B_Micro, J2 Conn_01x05_Female, J3 Conn_01x04_Female, J4 Conn_01x04_Female, SW1 SW_SPST, SW2 SW_Push, SW3 SW_Push, U1 ATtiny85V-10P

Commit message: UART 2 USB 4x1 socket turned by 180°, some traces rerouted -> simpler layout
Parts:
- moved J2 10.2 mm to (132.1, 101.6), turned to 0 degrees
Routing:
- net Earth: track 201.6 -> 183.8 mm
- net PB0: track 54.6 -> 52.8 mm, vias 0 -> 2
- net PB2: track 34.9 -> 33.8 mm
Changed lines of the file:
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@@
   )
   (footprint "Connector_PinSocket_2.54mm:PinSocket_1x05_P2.54mm_Vertical" (layer "F.Cu")
-    (at 132.08 111.76 180)
+    (at 132.08 101.6)
     (descr "Through hole straight socket strip, 1x05, 2.54mm pitch, single row (from Kicad 4.0.7), script generated")
     (tags "Through hole socket strip THT 1x05 2.54mm single row")
@@
     (fp_line (start 1.27 11.43) (end -1.27 11.43) (layer "F.Fab") (width 0.1))
     (fp_line (start 0.635 -1.27) (end 1.27 -0.635) (layer "F.Fab") (width 0.1))
-    (pad "1" thru_hole rect (at 0 0 180) (size 1.7 1.7) (drill 1) (layers *.Cu *.Mask)
+    (pad "1" thru_hole rect (at 0 0) (size 1.7 1.7) (drill 1) (layers *.Cu *.Mask)
       (net 10 "unconnected-(J2-Pad1)") (pinfunction "Pin_1") (pintype "passive+no_connect"))
-    (pad "2" thru_hole oval (at 0 2.54 180) (size 1.7 1.7) (drill 1) (layers *.Cu *.Mask)
+    (pad "2" thru_hole oval (at 0 2.54) (size 1.7 1.7) (drill 1) (layers *.Cu *.Mask)
       (net 11 "unconnected-(J2-Pad2)") (pinfunction "Pin_2") (pintype "passive+no_connect"))
-    (pad "3" thru_hole oval (at 0 5.08 180) (size 1.7 1.7) (drill 1) (layers *.Cu *.Mask)
+    (pad "3" thru_hole oval (at 0 5.08) (size 1.7 1.7) (drill 1) (layers *.Cu *.Mask)
       (net 12 "PB0") (pinfunction "Pin_3") (pintype "passive"))
-    (pad "4" thru_hole oval (at 0 7.62 180) (size 1.7 1.7) (drill 1) (layers *.Cu *.Mask)
+    (pad "4" thru_hole oval (at 0 7.62) (size 1.7 1.7) (drill 1) (layers *.Cu *.Mask)
       (net 13 "PB2") (pinfunction "Pin_4") (pintype "passive"))
-    (pad "5" thru_hole oval (at 0 10.16 180) (size 1.7 1.7) (drill 1) (layers *.Cu *.Mask)
+    (pad "5" thru_hole oval (at 0 10.16) (size 1.7 1.7) (drill 1) (layers *.Cu *.Mask)
       (net 9 "Earth") (pinfunction "Pin_5") (pintype "passive"))
     (model "${KICAD6_3DMODEL_DIR}/Connector_PinSocket_2.54mm.3dshapes/PinSocket_1x05_P2.54mm_Vertical.wrl"
@@
   (segment (start 101.6 96.52) (end 109.22 96.52) (width 0.25) (layer "F.Cu") (net 9))
   (segment (start 122.67 81.28) (end 137.16 81.28) (width 0.25) (layer "F.Cu") (net 9))
-  (segment (start 114.3 113.78) (end 114.3 129.54) (width 0.25) (layer "F.Cu") (net 9))
   (segment (start 106.99 78.74) (end 107.73 79.48) (width 0.25) (layer "F.Cu") (net 9))
-  (segment (start 109.22 111.76) (end 104.14 111.76) (width 0.25) (layer "F.Cu") (net 9))
+  (segment (start 132.08 111.76) (end 137.16 111.76) (width 0.25) (layer "F.Cu") (net 9))
   (segment (start 107.73 79.48) (end 120.87 79.48) (width 0.25) (layer "F.Cu") (net 9))
+  (segment (start 111.76 127) (end 109.22 127) (width 0.25) (layer "F.Cu") (net 9))
+  (segment (start 111.76 114.3) (end 111.76 127) (width 0.25) (layer "F.Cu") (net 9))
   (segment (start 137.16 91.44) (end 134.62 91.44) (width 0.25) (layer "F.Cu") (net 9))
   (segment (start 99.06 127) (end 104.14 127) (width 0.25) (layer "F.Cu") (net 9))
+  (segment (start 109.76 111.76) (end 111.02 110.5) (width 0.25) (layer "F.Cu") (net 9))
   (segment (start 99.06 120.65) (end 99.06 127) (width 0.25) (layer "F.Cu") (net 9))
   (segment (start 104.14 127) (end 109.22 127) (width 0.25) (layer "F.Cu") (net 9))
-  (segment (start 111.02 110.5) (end 114.3 113.78) (width 0.25) (layer "F.Cu") (net 9))
+  (segment (start 111.02 113.56) (end 111.76 114.3) (width 0.25) (layer "F.Cu") (net 9))
+  (segment (start 137.16 111.76) (end 137.16 96.52) (width 0.25) (layer "F.Cu") (net 9))
   (segment (start 133.35 96.52) (end 137.16 96.52) (width 0.25) (layer "F.Cu") (net 9))
   (segment (start 137.16 81.28) (end 137.16 91.44) (width 0.25) (layer "F.Cu") (net 9))
-  (segment (start 137.16 129.54) (end 137.16 96.52) (width 0.25) (layer "F.Cu") (net 9))
+  (segment (start 137.16 129.54) (end 137.16 111.76) (width 0.25) (layer "F.Cu") (net 9))
   (segment (start 101.6 78.74) (end 106.99 78.74) (width 0.25) (layer "F.Cu") (net 9))
   (segment (start 114.3 129.54) (end 137.16 129.54) (width 0.25) (layer "F.Cu") (net 9))
-  (segment (start 104.14 111.76) (end 104.14 127) (width 0.25) (layer "F.Cu") (net 9))
   (segment (start 120.87 79.48) (end 122.67 81.28) (width 0.25) (layer "F.Cu") (net 9))
   (segment (start 137.16 96.52) (end 137.16 91.44) (width 0.25) (layer "F.Cu") (net 9))
-  (segment (start 111.02 110.5) (end 109.76 111.76) (width 0.25) (layer "F.Cu") (net 9))
-  (segment (start 109.76 111.76) (end 109.22 111.76) (width 0.25) (layer "F.Cu") (net 9))
-  (segment (start 132.08 101.6) (end 137.16 101.6) (width 0.25) (layer "F.Cu") (net 9))
+  (segment (start 111.76 127) (end 114.3 129.54) (width 0.25) (layer "F.Cu") (net 9))
+  (segment (start 111.02 110.5) (end 111.02 113.56) (width 0.25) (layer "F.Cu") (net 9))
+  (segment (start 109.22 111.76) (end 109.76 111.76) (width 0.25) (layer "F.Cu") (net 9))
   (via (at 109.22 111.76) (size 0.8) (drill 0.4) (layers "F.Cu" "B.Cu") (net 9))
   (via (at 109.22 96.52) (size 0.8) (drill 0.4) (layers "F.Cu" "B.Cu") (net 9))
   (segment (start 109.22 111.76) (end 109.22 96.52) (width 0.25) (layer "B.Cu") (net 9))
   (segment (start 129.54 106.68) (end 132.08 106.68) (width 0.25) (layer "F.Cu") (net 12))
+  (segment (start 116.84 127) (end 119.38 127) (width 0.25) (layer "F.Cu") (net 12))
+  (segment (start 116.84 112.3) (end 116.84 127) (width 0.25) (layer "F.Cu") (net 12))
+  (segment (start 118.64 110.5) (end 116.84 112.3) (width 0.25) (layer "F.Cu") (net 12))
   (segment (start 124.46 127) (end 129.54 127) (width 0.25) (layer "F.Cu") (net 12))
   (segment (start 124.46 127) (end 119.38 127) (width 0.25) (layer "F.Cu") (net 12))
-  (segment (start 118.64 110.5) (end 120.66 110.5) (width 0.25) (layer "F.Cu") (net 12))
-  (segment (start 129.54 127) (end 129.54 106.68) (width 0.25) (layer "F.Cu") (net 12))
-  (segment (start 121.92 111.76) (end 124.46 111.76) (width 0.25) (layer "F.Cu") (net 12))
-  (segment (start 124.46 111.76) (end 124.46 127) (width 0.25) (layer "F.Cu") (net 12))
-  (segment (start 120.66 110.5) (end 121.92 111.76) (width 0.25) (layer "F.Cu") (net 12))
+  (segment (start 129.54 127) (end 129.54 111.76) (width 0.25) (layer "F.Cu") (net 12))
+  (via (at 129.54 111.76) (size 0.8) (drill 0.4) (layers "F.Cu" "B.Cu") (net 12))
+  (via (at 129.54 106.68) (size 0.8) (drill 0.4) (layers "F.Cu" "B.Cu") (net 12))
+  (segment (start 129.54 111.76) (end 129.54 106.68) (width 0.25) (layer "B.Cu") (net 12))
   (segment (start 118.64 105.42) (end 125.74 105.42) (width 0.25) (layer "F.Cu") (net 13))
-  (segment (start 129.54 104.14) (end 132.08 104.14) (width 0.25) (layer "F.Cu") (net 13))
   (segment (start 119.38 121.92) (end 121.92 121.92) (width 0.25) (layer "F.Cu") (net 13))
-  (segment (start 127 106.68) (end 129.54 104.14) (width 0.25) (layer "F.Cu") (net 13))
+  (segment (start 127 109.22) (end 132.08 109.22) (width 0.25) (layer "F.Cu") (net 13))
   (segment (start 125.74 105.42) (end 127 106.68) (width 0.25) (layer "F.Cu") (net 13))
+  (segment (start 127 106.68) (end 127 109.22) (width 0.25) (layer "F.Cu") (net 13))
+  (via (at 127 109.22) (size 0.8) (drill 0.4) (layers "F.Cu" "B.Cu") (net 13))
   (via (at 121.92 121.92) (size 0.8) (drill 0.4) (layers "F.Cu" "B.Cu") (net 13))
-  (via (at 127 106.68) (size 0.8) (drill 0.4) (layers "F.Cu" "B.Cu") (net 13))
-  (segment (start 127 106.68) (end 127 116.84) (width 0.25) (layer "B.Cu") (net 13))
   (segment (start 127 116.84) (end 121.92 121.92) (width 0.25) (layer "B.Cu") (net 13))
+  (segment (start 127 109.22) (end 127 116.84) (width 0.25) (layer "B.Cu") (net 13))
   (segment (start 109.22 119.38) (end 106.68 119.38) (width 0.25) (layer "F.Cu") (net 14))
   (segment (start 111.02 102.88) (end 107.94 102.88) (width 0.25) (layer "F.Cu") (net 14))
